Commit message: xacro functions

File: ros2_workspace/src/my_robot_description/urdf/first_robot.urdf.xacro (robot description, xacro)
@@ -6,4 +6,15 @@
     <xacro:property name="wheel_radius" value="0.1" />
     <xacro:property name="wheel_length" value="0.05" />
+    <xacro:macro name="wheel_link" params="prefix">
+        <link name="${prefix}_wheel_link">
+            <visual>
+                <geometry>
+                    <cylinder radius="${wheel_radius}" length="${wheel_length}" />
+                </geometry>
+                <origin xyz="0 0 0" rpy="${pi / 2.0} 0 0" />
+                <material name="grey" />
+            </visual>
+        </link>
+    </xacro:macro>
     <material name="green">
         <color rgba="0 0.5 0 1" />
@@ -25,22 +36,6 @@
         </visual>
     </link>
-    <link name="right_wheel_link">
-        <visual>
-            <geometry>
-                <cylinder radius="${wheel_radius}" length="${wheel_length}" />
-            </geometry>
-            <origin xyz="0 0 0" rpy="${pi / 2.0} 0 0" />
-            <material name="grey" />
-        </visual>
-    </link>
-    <link name="left_wheel_link">
-        <visual>
-            <geometry>
-                <cylinder radius="${wheel_radius}" length="${wheel_length}" />
-            </geometry>
-            <origin xyz="0 0 0" rpy="${pi / 2.0} 0 0" />
-            <material name="grey" />
-        </visual>
-    </link>
+    <xacro:wheel_link prefix="right" />
+    <xacro:wheel_link prefix="left" />
     <link name="cluster_wheel_link">
         <visual>

Commit message: Include a Xacro File in Another Xacro File

File: ros2_workspace/src/my_robot_description/urdf/first_robot.urdf.xacro (robot description, xacro)
@@ -1,71 +1,5 @@
 <?xml version="1.0"?>
 <robot name="first_robot" xmlns:xacro="http://www.ros.org/wiki/xacro">
-    <xacro:property name="base_length" value="0.6" />
-    <xacro:property name="base_width" value="0.4" />
-    <xacro:property name="base_height" value="0.2" />
-    <xacro:property name="wheel_radius" value="0.1" />
-    <xacro:property name="wheel_length" value="0.05" />
-    <xacro:macro name="wheel_link" params="prefix">
-        <link name="${prefix}_wheel_link">
-            <visual>
-                <geometry>
-                    <cylinder radius="${wheel_radius}" length="${wheel_length}" />
-                </geometry>
-                <origin xyz="0 0 0" rpy="${pi / 2.0} 0 0" />
-                <material name="grey" />
-            </visual>
-        </link>
-    </xacro:macro>
-    <material name="green">
-        <color rgba="0 0.5 0 1" />
-    </material>
-    <material name="blue">
-        <color rgba="0 0 0.5 1" />
-    </material>
-    <material name="grey">
-        <color rgba="0.5 0.5 0.5 1" />
-    </material>
-    <link name="base_footprint" />
-    <link name="base_link">
-        <visual>
-            <geometry>
-                <box size="${base_length} ${base_width} ${base_height}" />
-            </geometry>
-            <origin xyz="0 0 0.1" rpy="0 0 0" />
-            <material name="blue" />
-        </visual>
-    </link>
-    <xacro:wheel_link prefix="right" />
-    <xacro:wheel_link prefix="left" />
-    <link name="cluster_wheel_link">
-        <visual>
-            <geometry>
-                <sphere radius="${wheel_length}" />
-            </geometry>
-            <origin xyz="0 0 0" rpy="0 0 0" />
-            <material name="grey" />
-        </visual>
-    </link>
-    <joint name="base_footprint_joint" type="fixed">
-        <parent link="base_footprint" />
-        <child link="base_link" />
-        <origin xyz="0 0 0.1" rpy="0 0 0" />
-    </joint>
-    <joint name="base_right_wheel_joint" type="continuous">
-        <parent link="base_link" />
-        <child link="right_wheel_link" />
-        <origin xyz="${-base_length / 4.0}  ${- base_width / 2 - wheel_length / 2 } 0" rpy="0 0 0" />
-        <axis xyz="0 1 0.0" />
-    </joint>
-    <joint name="base_left_wheel_joint" type="continuous">
-        <parent link="base_link" />
-        <child link="left_wheel_link" />
-        <origin xyz="${-base_length / 4.0} ${base_width / 2 + wheel_length / 2} 0" rpy="0 0 0" />
-        <axis xyz="0 1 0.0" />
-    </joint>
-    <joint name="base_cluster_wheel_joint" type="fixed">
-        <parent link="base_link" />
-        <child link="cluster_wheel_link" />
-        <origin xyz="${base_length / 3} 0 ${-wheel_length}" rpy="0 0 0" />
-    </joint>
+    <xacro:include filename="common.properties.xacro" />
+    <xacro:include filename="mobile.base.xacro" />
 </robot>
